File: schematics/Z8C rev3/file62109D9A.sch (KiCad schematic (older format))
At the start: 7 parts

Commit message: added bank switching, apu, dma and IRQ logic. Misc. improvements
Parts:
- removed U?: Si5351A-B-GT, Package_SO:MSOP-10_3x3mm_P0.5mm, symbol Oscillator:Si5351A-B-GT
- U37: renamed from U?; symbol ym2612:YM2612 -> Z8C-rev3-rescue:YM2612-ym2612
- U40: renamed from U?; symbol oldchips:AY-3-8912 -> Z8C-rev3-rescue:AY-3-8912-oldchips
- U41: renamed from U?; symbol audio_tk:SN76489AN -> Z8C-rev3-rescue:SN76489AN-audio_tk
- gave numbers to parts that had none: 2
Changed lines of the file:
@@
 $Descr A4 11693 8268
 encoding utf-8
-Sheet 7 7
+Sheet 6 7
 Title ""
 Date ""
@@
 $EndDescr
 $Comp
-L ym2612:YM2612 U?
+L Z8C-rev3-rescue:YM2612-ym2612 U37
 U 1 1 6210A0AA
 P 2850 3250
-F 0 "U?" H 3200 4037 60  0000 C CNN
+F 0 "U37" H 3200 4037 60  0000 C CNN
 F 1 "YM2612" H 3200 3931 60  0000 C CNN
 F 2 "" H 3200 4000 60  0001 C CNN
 F 3 "" H 3200 4000 60  0001 C CNN
 	1    2850 3250
-	1    0    0    -1
-$EndComp
-$Comp
-L Oscillator:Si5351A-B-GT U?
-U 1 1 6210B43C
-P 3200 1300
-F 0 "U?" H 2900 1750 50  0000 C CNN
-F 1 "Si5351A-B-GT" H 3550 800 50  0000 C CNN
-F 2 "Package_SO:MSOP-10_3x3mm_P0.5mm" H 3200 500 50  0001 C CNN
-F 3 "https://www.silabs.com/documents/public/data-sheets/Si5351-B.pdf" H 2850 1200 50  0001 C CNN
-	1    3200 1300
 	1    0    0    -1
 $EndComp
@@
 	2300 3750 2650 3750
 $Comp
-L power:GND #PWR?
+L power:GND #PWR0143
 U 1 1 6211B340
 P 2550 3950
-F 0 "#PWR?" H 2550 3700 50  0001 C CNN
+F 0 "#PWR0143" H 2550 3700 50  0001 C CNN
 F 1 "GND" H 2555 3777 50  0000 C CNN
 F 2 "" H 2550 3950 50  0001 C CNN
@@
 Connection ~ 2550 3850
 $Comp
-L power:GND #PWR?
+L power:GND #PWR0144
 U 1 1 6211D42B
 P 3950 3900
-F 0 "#PWR?" H 3950 3650 50  0001 C CNN
+F 0 "#PWR0144" H 3950 3650 50  0001 C CNN
 F 1 "GND" H 3955 3727 50  0000 C CNN
 F 2 "" H 3950 3900 50  0001 C CNN
@@
 	3950 3250 3750 3250
 $Comp
-L power:+5V #PWR?
+L power:+5V #PWR0145
 U 1 1 6211DE8B
 P 3850 2600
-F 0 "#PWR?" H 3850 2450 50  0001 C CNN
+F 0 "#PWR0145" H 3850 2450 50  0001 C CNN
 F 1 "+5V" H 3865 2773 50  0000 C CNN
 F 2 "" H 3850 2600 50  0001 C CNN
@@
 Connection ~ 3850 2850
 $Comp
-L audio_tk:SN76489AN U?
+L Z8C-rev3-rescue:SN76489AN-audio_tk U41
 U 1 1 62123F49
 P 5600 3300
-F 0 "U?" H 5600 4175 50  0000 C CNN
+F 0 "U41" H 5600 4175 50  0000 C CNN
 F 1 "SN76489AN" H 5600 4084 50  0000 C CNN
 F 2 "Package_DIP:DIP-16_W7.62mm" H 5600 3300 50  0001 C CNN
@@
 NoConn ~ 3750 3850
 $Comp
-L oldchips:AY-3-8912 U?
+L Z8C-rev3-rescue:AY-3-8912-oldchips U40
 U 1 1 62135F28
 P 5200 4600
-F 0 "U?" H 5600 4765 50  0000 C CNN
+F 0 "U40" H 5600 4765 50  0000 C CNN
 F 1 "AY-3-8912" H 5600 4674 50  0000 C CNN
 F 2 "oldchips-DIL40" H 5200 4750 50  0001 C CNN
@@
 NoConn ~ 5000 5500
 $Comp
-L power:+5V #PWR?
+L power:+5V #PWR0146
 U 1 1 62143E89
 P 4800 5700
-F 0 "#PWR?" H 4800 5550 50  0001 C CNN
+F 0 "#PWR0146" H 4800 5550 50  0001 C CNN
 F 1 "+5V" H 4815 5873 50  0000 C CNN
 F 2 "" H 4800 5700 50  0001 C CNN
@@
 CS_AY
 $Comp
-L 74xx:74LS08 U?
+L 74xx:74LS08 U39
 U 1 1 6214F51B
 P 3700 5300
-F 0 "U?" H 3700 5625 50  0000 C CNN
+F 0 "U39" H 3700 5625 50  0000 C CNN
 F 1 "74LS08" H 3700 5534 50  0000 C CNN
 F 2 "" H 3700 5300 50  0001 C CNN
@@
 $EndComp
 $Comp
-L 74xx:74LS08 U?
+L 74xx:74LS08 U39
 U 2 1 62152BB2
 P 3700 6000
-F 0 "U?" H 3700 6325 50  0000 C CNN
+F 0 "U39" H 3700 6325 50  0000 C CNN
 F 1 "74LS08" H 3700 6234 50  0000 C CNN
 F 2 "" H 3700 6000 50  0001 C CNN
@@
 	3150 5200 3150 4750
 $Comp
-L 74xx:74HC04 U?
+L 74xx:74HC04 U38
 U 1 1 6215FD1D
 P 2900 6100
-F 0 "U?" H 2900 6417 50  0000 C CNN
+F 0 "U38" H 2900 6417 50  0000 C CNN
 F 1 "74HC04" H 2900 6326 50  0000 C CNN
 F 2 "" H 2900 6100 50  0001 C CNN
@@
 Wire Bus Line
 	2700 4400 1950 4400
-$Comp
-L power:+3.3V #PWR?
-U 1 1 62211364
-P 3100 750
-F 0 "#PWR?" H 3100 600 50  0001 C CNN
-F 1 "+3.3V" H 3115 923 50  0000 C CNN
-F 2 "" H 3100 750 50  0001 C CNN
-F 3 "" H 3100 750 50  0001 C CNN
-	1    3100 750
-	1    0    0    -1
-$EndComp
-$Comp
-L power:GND #PWR?
-U 1 1 622121B8
-P 3200 1900
-F 0 "#PWR?" H 3200 1650 50  0001 C CNN
-F 1 "GND" H 3205 1727 50  0000 C CNN
-F 2 "" H 3200 1900 50  0001 C CNN
-F 3 "" H 3200 1900 50  0001 C CNN
-	1    3200 1900
-	1    0    0    -1
-$EndComp
-Wire Wire Line
-	3200 1900 3200 1800
-Wire Wire Line
-	3100 800  3100 750
-Wire Wire Line
-	3100 750  3300 750
-Wire Wire Line
-	3300 750  3300 800
 Wire Bus Line
 	4450 2750 4450 4400
@@
 Wire Bus Line
 	1950 2750 1950 4400
-Connection ~ 3100 750
 $EndSCHEMATC
