File: schematics/Z8C rev3/file622409DB.sch (KiCad schematic (older format))
At the start: 15 parts

Commit message: added bank switching, apu, dma and IRQ logic. Misc. improvements
Parts:
- removed U?: 74HC154, symbol 74xx:74LS154
- added J5: DIN-5, symbol Connector:DIN-5
- added U31: PIO-DIP-40, Package_DIP:DIP-40_W15.24mm, symbol Z8C-rev3-rescue:PIO-DIP-40-Zilog_Z80_Peripherals
- added U32, U33: 74HC595, Package_DIP:DIP-14_W7.62mm_LongPads, symbol 74xx:74HC595
- added U34: 74HC125, Package_DIP:DIP-14_W7.62mm_LongPads, symbol 74xx:74LS125
- IC1: renamed from IC?; symbol Zilog_Z80_Peripherals:CTC-DIP-28 -> Z8C-rev3-rescue:CTC-DIP-28-Zilog_Z80_Peripherals
- IC2: renamed from IC?; symbol Zilog_Z80_Peripherals:SIO0-DIP-40 -> Z8C-rev3-rescue:SIO0-DIP-40-Zilog_Z80_Peripherals
- U35, U36: renamed from U?; footprint (none) -> Package_DIP:DIP-14_W7.62mm_LongPads
- gave numbers to parts that had none: 10
Connections:
- net !INT: now also U31.23 (~INT~)
- net !IOREQ: now also U31.36 (~IORQ~)
- net !M1: now also U31.37 (~M1~)
- net !RD: now also U31.35 (~RD~)
- net A0: now also U31.5 (C/~D~)
- net A1: now also U31.6 (B/~A~)
- net CLK_CPU: now also U31.25 (CLK)
- net GND: now also J5.2, U32.13 (~OE), U33.13 (~OE)
- net at IC1.11 (IEO): now also IC1.7 (ZC/TO0), IC2.13 (~RXCA), IC2.14 (~TXCA); no longer IC2.6 (IEI)
- net CS_CTC renamed IO_CTC_CS
- net CS_SIO renamed IO_SIO_CS
- net RESET renamed !RESET
- new net: U31.8 (PA6), U32.7 (QH)
- new net: U32.9 (QH'), U33.14 (SER)
- new net +5V: J5.1
- new net CLEAR: U31.29 (PB2), U32.10 (~SRCLR), U33.10 (~SRCLR)
- new net DATA0: U31.15 (PA0), U32.1 (QB)
- new net DATA1: U31.14 (PA1), U32.2 (QC)
- new net DATA2: U31.13 (PA2), U32.3 (QD)
- new net DATA3: U31.12 (PA3), U32.4 (QE)
- new net DATA5: U31.10 (PA4), U32.5 (QF)
- new net DATA6: U31.9 (PA5), U32.6 (QG)
- new net DATA7: U31.7 (PA7), U33.15 (QA)
- new net IO_PS2_CS: U31.4 (~CE~)
- new net PARITY: U31.27 (PB0), U33.1 (QB)
- new net PS2_CLK: J5.5, U32.11 (SRCLK), U32.12 (RCLK), U33.11 (SRCLK), U33.12 (RCLK), U34.6
- new net PS2_DATA: J5.4, U32.14 (SER), U34.3
- new net SCLK: U31.31 (PB4), U34.5
- new net SDATA: U31.30 (PB3), U34.2
- new net SENABLE: U31.32 (PB5), U34.1, U34.4
- new net STOP: U31.28 (PB1), U33.2 (QC)
- no-connect marks 9 -> 13
Other:
- moved on the sheet: C10, C11, C12, C13, C14, C15, C16, C9, IC1, IC2, J6, J7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
